Commit message: lio-sam mapping

File: robots/a1_description/xacro/robot.xacro (robot description, xacro)
@@ -14,11 +14,11 @@
     <xacro:if value="$(arg DEBUG)">
         <link name="world"/>
-        <joint name="base_static_joint" type="fixed">
+        <joint name="base_link_static_joint" type="fixed">
             <origin rpy="0 0 0" xyz="0 0 0"/>
             <parent link="world"/>
-            <child link="base"/>
+            <child link="base_link"/>
         </joint>
     </xacro:if>
-    <link name="base">
+    <link name="base_link">
         <visual>
             <origin rpy="0 0 0" xyz="0 0 0"/>
@@ -28,7 +28,15 @@
         </visual>
     </link>
-    <joint name="floating_base" type="fixed">
+    <xacro:arg name="gpu" default="false"/>
+    <xacro:property name="gpu" value="$(arg gpu)" />
+    <xacro:arg name="organize_cloud" default="false"/>
+    <xacro:property name="organize_cloud" value="$(arg organize_cloud)" />
+    <xacro:include filename="$(find velodyne_description)/urdf/VLP-16.urdf.xacro"/>
+    <xacro:VLP-16 parent="base_link" name="velodyne" topic="/velodyne_points" organize_cloud="${organize_cloud}" hz="10" samples="440" gpu="${gpu}">
+        <origin xyz="0 0 0.07" rpy="0 0 0" />
+    </xacro:VLP-16>
+    <joint name="floating_base_link" type="fixed">
         <origin rpy="0 0 0" xyz="0 0 0"/>
-        <parent link="base"/>
+        <parent link="base_link"/>
         <child link="trunk"/>
     </joint>
